File: Hardware/FrontPanel.sch (EAGLE design)
At the start: 24 parts, among them U1 TPIC6B595N, U2 TPIC6B595N, U3 TPIC6B595N, U4 TPIC6B595N, U5 TPIC6B595N, U6 TPIC6B595N

Commit message: fixed ERC errors
Parts:
- D1, D2: value (none) -> RED/AMBER; device Wurth_Elektronik_Optoelectronics_rev17b:WL-SMTW_3528-150141AS73100-A -> Wurth_Elektronik_Optoelectronics_rev18a:WL-SITW_3528_15414185BA210
- DATA, HV: value (none) -> .1" Header
Connections:
- net +160V renamed V+
- net +5V renamed VCC
- net GND: now also U1.GND, U2.GND, U3.GND, U4.GND, U5.GND, U6.GND; no longer U1.GND1, U1.GND2, U1.GND3, U2.GND1, U2.GND2, U2.GND3, U3.GND1, U3.GND2, U3.GND3, U4.GND1, U4.GND2, U4.GND3, U5.GND1, U5.GND2, U5.GND3, U6.GND1, U6.GND2, U6.GND3
