File: Hardware/Panel.brd (EAGLE design)
At the start: 100 x 100 mm, 44 parts, among them IC1 74HCT04D, U1 TPIC6B595N, U2 TPIC6B595N, U3 TPIC6B595N, U4 TPIC6B595N, U5 TPIC6B595N, U6 TPIC6B595N, U7 CJT1117-3.3-SOT223

Commit message: fixed ERC errors
Parts:
- D1, D2: value (none) -> RED/AMBER; device Wurth_Elektronik_Optoelectronics_rev17b:WL-SMTW_3528 -> Wurth_Elektronik_Optoelectronics_rev18a:WL-SITW_154141XXBA210
- DATA, HV: value (none) -> .1" Header
- turned D1 to 180 degrees
- turned D2 to 180 degrees
Connections:
- net +160V renamed V+
- removed net +5V1: C2.1, DATA1.1, IC1.14, U$12.5V, U7.2, U7.TER
- new net VCC: DATA.5, R10.2, R9.2, U1.2, U1.8, U2.2, U2.8, U3.2, U3.8, U4.2, U4.8, U5.2, U5.8, U6.2, U6.8
- net +5V: now also C2.1, DATA1.1, IC1.14, U$12.5V, U7.2, U7.TER; no longer DATA.5, R10.2, R9.2, U1.2, U1.8, U2.2, U2.8, U3.2, U3.8, U4.2, U4.8, U5.2, U5.8, U6.2, U6.8
- net LED1: now also D1.2; no longer D1.1
- net LED2: now also D2.2; no longer D2.1
- net N$66: now also D1.1; no longer D1.2
- net N$67: now also D2.1; no longer D2.2
Routing:
- net VCC: track 0.00 -> 280.9 mm, vias 0 -> 8
- net +5V: track 280.9 -> 61.9 mm, vias 8 -> 0
- net +5V1: track 61.9 -> 0.00 mm
- net GND: track 79.0 -> 64.4 mm
